File: pcb/target/esd_power.kicad_sch (KiCad schematic)
At the start: 1 part

Commit message: redid target pcb with new components
Connections:
- net GND Main: now also D19.1 (A1); no longer D19.2 (A2)
- net IN: now also D19.2 (A2); no longer D19.1 (A1)
Other:
- moved on the sheet: D19
Changed lines of the file:
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@@
 	(symbol
 		(lib_id "Diode:SMAJ6.0CA")
-		(at 76.2 85.09 270)
+		(at 76.2 85.09 90)
 		(unit 1)
 		(exclude_from_sim no)
@@
 					(size 1.27 1.27)
 				)
-				(justify left)
+				(justify right)
 			)
 		)
@@
 					(size 1.27 1.27)
 				)
-				(justify left)
+				(justify right)
 			)
 		)
 		(property "Footprint" "Diode_SMD:D_SMA"
-			(at 71.12 85.09 0)
+			(at 81.28 85.09 0)
 			(effects
 				(font
