File: pcb/target/led.kicad_sch (KiCad schematic)
At the start: 4 parts, among them J8 Conn_01x03_Pin, J9 Conn_01x03_Pin

Commit message: finishing up target pcb
Parts:
- J8, J9: footprint Connector_Wire:SolderWire-0.25sqmm_1x03_P4.2mm_D0.65mm_OD1.7mm -> custom_footprints:01x03 SMD 2x3mm pad
Changed lines of the file:
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@@
 			)
 		)
-		(property "Footprint" "Connector_Wire:SolderWire-0.25sqmm_1x03_P4.2mm_D0.65mm_OD1.7mm"
+		(property "Footprint" "custom_footprints:01x03 SMD 2x3mm pad"
 			(at 175.26 58.42 0)
 			(effects
@@
 			)
 		)
-		(property "Footprint" "Connector_Wire:SolderWire-0.25sqmm_1x03_P4.2mm_D0.65mm_OD1.7mm"
+		(property "Footprint" "custom_footprints:01x03 SMD 2x3mm pad"
 			(at 74.93 58.42 0)
 			(effects

Commit message: added lcsc numbers to all components and added ESD protection
Parts:
- D6, D7: LCSC (none) -> C5349959
Changed lines of the file:
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@@
+			)
+		)
+		(property "LCSC" "C5349959"
+			(at 95.25 58.42 0)
+			(effects
+				(font
+					(size 1.27 1.27)
+				)
+				(hide yes)
 			)
 		)
@@
 		(instances
 			(project "target"
-				(path "/1c02f793-f381-44cb-838a-dbb787484d0c/e61b723f-f359-4114-beb0-b4d2930b2aa9/57687f76-c606-4b93-8b3a-c2df1794cc42"
-					(reference "D8")
-					(unit 1)
-				)
-				(path "/1c02f793-f381-44cb-838a-dbb787484d0c/e61b723f-f359-4114-beb0-b4d2930b2aa9/59431009-1e31-4aed-9634-5b986cfe3fa7"
+				(path "/1c02f793-f381-44cb-838a-dbb787484d0c/e61b723f-f359-4114-beb0-b4d2930b2aa9/34d9b2fa-eed6-45bc-971e-9a5c863f1de0"
 					(reference "D14")
 					(unit 1)
 				)
-				(path "/1c02f793-f381-44cb-838a-dbb787484d0c/e61b723f-f359-4114-beb0-b4d2930b2aa9/909bdbb4-b84d-4035-be27-26a2c2c664d8"
-					(reference "D12")
+				(path "/1c02f793-f381-44cb-838a-dbb787484d0c/e61b723f-f359-4114-beb0-b4d2930b2aa9/611ab34e-dc39-47a6-a008-28f4f9825563"
+					(reference "D2")
 					(unit 1)
 				)
 				(path "/1c02f793-f381-44cb-838a-dbb787484d0c/e61b723f-f359-4114-beb0-b4d2930b2aa9/f47d6d41-3ee7-4ca5-8055-90d1df9d67d0"
 					(reference "D6")
+					(unit 1)
+				)
+				(path "/1c02f793-f381-44cb-838a-dbb787484d0c/e61b723f-f359-4114-beb0-b4d2930b2aa9/fcf601a2-49b1-4c8c-9ec7-cdc985204443"
+					(reference "D10")
 					(unit 1)
 				)
@@
 			)
 		)
+		(property "LCSC" "C5349959"
+			(at 133.35 58.42 0)
+			(effects
+				(font
+					(size 1.27 1.27)
+				)
+				(hide yes)
+			)
+		)
 		(pin "6"
 		)
@@
 		(instances
 			(project "target"
-				(path "/1c02f793-f381-44cb-838a-dbb787484d0c/e61b723f-f359-4114-beb0-b4d2930b2aa9/57687f76-c606-4b93-8b3a-c2df1794cc42"
-					(reference "D9")
-					(unit 1)
-				)
-				(path "/1c02f793-f381-44cb-838a-dbb787484d0c/e61b723f-f359-4114-beb0-b4d2930b2aa9/59431009-1e31-4aed-9634-5b986cfe3fa7"
+				(path "/1c02f793-f381-44cb-838a-dbb787484d0c/e61b723f-f359-4114-beb0-b4d2930b2aa9/34d9b2fa-eed6-45bc-971e-9a5c863f1de0"
 					(reference "D15")
 					(unit 1)
 				)
-				(path "/1c02f793-f381-44cb-838a-dbb787484d0c/e61b723f-f359-4114-beb0-b4d2930b2aa9/909bdbb4-b84d-4035-be27-26a2c2c664d8"
-					(reference "D13")
+				(path "/1c02f793-f381-44cb-838a-dbb787484d0c/e61b723f-f359-4114-beb0-b4d2930b2aa9/611ab34e-dc39-47a6-a008-28f4f9825563"
+					(reference "D3")
 					(unit 1)
 				)
 				(path "/1c02f793-f381-44cb-838a-dbb787484d0c/e61b723f-f359-4114-beb0-b4d2930b2aa9/f47d6d41-3ee7-4ca5-8055-90d1df9d67d0"
 					(reference "D7")
+					(unit 1)
+				)
+				(path "/1c02f793-f381-44cb-838a-dbb787484d0c/e61b723f-f359-4114-beb0-b4d2930b2aa9/fcf601a2-49b1-4c8c-9ec7-cdc985204443"
+					(reference "D11")
 					(unit 1)
 				)
@@
 			)
 		)
+		(property "LCSC" ""
+			(at 175.26 58.42 0)
+			(effects
+				(font
+					(size 1.27 1.27)
+				)
+				(hide yes)
+			)
+		)
 		(pin "3"
 		)
@@
 		(instances
 			(project "target"
-				(path "/1c02f793-f381-44cb-838a-dbb787484d0c/e61b723f-f359-4114-beb0-b4d2930b2aa9/57687f76-c606-4b93-8b3a-c2df1794cc42"
+				(path "/1c02f793-f381-44cb-838a-dbb787484d0c/e61b723f-f359-4114-beb0-b4d2930b2aa9/34d9b2fa-eed6-45bc-971e-9a5c863f1de0"
+					(reference "J19")
+					(unit 1)
+				)
+				(path "/1c02f793-f381-44cb-838a-dbb787484d0c/e61b723f-f359-4114-beb0-b4d2930b2aa9/611ab34e-dc39-47a6-a008-28f4f9825563"
 					(reference "J11")
-					(unit 1)
-				)
-				(path "/1c02f793-f381-44cb-838a-dbb787484d0c/e61b723f-f359-4114-beb0-b4d2930b2aa9/59431009-1e31-4aed-9634-5b986cfe3fa7"
-					(reference "J17")
-					(unit 1)
-				)
-				(path "/1c02f793-f381-44cb-838a-dbb787484d0c/e61b723f-f359-4114-beb0-b4d2930b2aa9/909bdbb4-b84d-4035-be27-26a2c2c664d8"
-					(reference "J15")
 					(unit 1)
 				)
 				(path "/1c02f793-f381-44cb-838a-dbb787484d0c/e61b723f-f359-4114-beb0-b4d2930b2aa9/f47d6d41-3ee7-4ca5-8055-90d1df9d67d0"
 					(reference "J9")
+					(unit 1)
+				)
+				(path "/1c02f793-f381-44cb-838a-dbb787484d0c/e61b723f-f359-4114-beb0-b4d2930b2aa9/fcf601a2-49b1-4c8c-9ec7-cdc985204443"
+					(reference "J15")
 					(unit 1)
 				)
@@
 			)
 		)
+		(property "LCSC" ""
+			(at 74.93 58.42 0)
+			(effects
+				(font
+					(size 1.27 1.27)
+				)
+				(hide yes)
+			)
+		)
 		(pin "3"
 		)
@@
 		(instances
 			(project "target"
-				(path "/1c02f793-f381-44cb-838a-dbb787484d0c/e61b723f-f359-4114-beb0-b4d2930b2aa9/57687f76-c606-4b93-8b3a-c2df1794cc42"
+				(path "/1c02f793-f381-44cb-838a-dbb787484d0c/e61b723f-f359-4114-beb0-b4d2930b2aa9/34d9b2fa-eed6-45bc-971e-9a5c863f1de0"
+					(reference "J18")
+					(unit 1)
+				)
+				(path "/1c02f793-f381-44cb-838a-dbb787484d0c/e61b723f-f359-4114-beb0-b4d2930b2aa9/611ab34e-dc39-47a6-a008-28f4f9825563"
 					(reference "J10")
-					(unit 1)
-				)
-				(path "/1c02f793-f381-44cb-838a-dbb787484d0c/e61b723f-f359-4114-beb0-b4d2930b2aa9/59431009-1e31-4aed-9634-5b986cfe3fa7"
-					(reference "J16")
-					(unit 1)
-				)
-				(path "/1c02f793-f381-44cb-838a-dbb787484d0c/e61b723f-f359-4114-beb0-b4d2930b2aa9/909bdbb4-b84d-4035-be27-26a2c2c664d8"
-					(reference "J14")
 					(unit 1)
 				)
@@
 					(unit 1)
 				)
+				(path "/1c02f793-f381-44cb-838a-dbb787484d0c/e61b723f-f359-4114-beb0-b4d2930b2aa9/fcf601a2-49b1-4c8c-9ec7-cdc985204443"
+					(reference "J14")
+					(unit 1)
+				)

Commit message: finished all pcbs by adjusting traces acording to 1oz copper weight
Parts:
- J8, J9: now left out of the parts list
Changed lines of the file:
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@@
 		(unit 1)
 		(exclude_from_sim no)
-		(in_bom yes)
+		(in_bom no)
 		(on_board yes)
 		(dnp no)
@@
 		(unit 1)
 		(exclude_from_sim no)
-		(in_bom yes)
+		(in_bom no)
 		(on_board yes)
 		(dnp no)
