File: pcb/target/led_cap.kicad_sch (KiCad schematic)
At the start: 5 parts, among them J6 Conn_01x03_Pin, J7 Conn_01x03_Pin

Commit message: finishing up target pcb
Parts:
- J6, J7: footprint Connector_Wire:SolderWire-0.25sqmm_1x03_P4.2mm_D0.65mm_OD1.7mm -> custom_footprints:01x03 SMD 2x3mm pad
Changed lines of the file:
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@@
 			)
 		)
-		(property "Footprint" "Connector_Wire:SolderWire-0.25sqmm_1x03_P4.2mm_D0.65mm_OD1.7mm"
+		(property "Footprint" "custom_footprints:01x03 SMD 2x3mm pad"
 			(at 67.31 50.8 0)
 			(effects
@@
 			)
 		)
-		(property "Footprint" "Connector_Wire:SolderWire-0.25sqmm_1x03_P4.2mm_D0.65mm_OD1.7mm"
+		(property "Footprint" "custom_footprints:01x03 SMD 2x3mm pad"
 			(at 181.61 50.8 0)
 			(effects

Commit message: added lcsc numbers to all components and added ESD protection
Parts:
- C2: LCSC (none) -> C93194
- D4, D5: LCSC (none) -> C5349959
Changed lines of the file:
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@@
+			)
+		)
+		(property "LCSC" "C93194"
+			(at 91.44 50.8 0)
+			(effects
+				(font
+					(size 1.27 1.27)
+				)
+				(hide yes)
 			)
 		)
@@
 		(instances
 			(project "target"
-				(path "/1c02f793-f381-44cb-838a-dbb787484d0c/e61b723f-f359-4114-beb0-b4d2930b2aa9/560cd6ce-e08c-4984-ad6c-35893396417e"
+				(path "/1c02f793-f381-44cb-838a-dbb787484d0c/e61b723f-f359-4114-beb0-b4d2930b2aa9/2577de81-7bff-4af3-a196-645474f5bc39"
 					(reference "C3")
 					(unit 1)
 				)
-				(path "/1c02f793-f381-44cb-838a-dbb787484d0c/e61b723f-f359-4114-beb0-b4d2930b2aa9/7ee20812-a607-4ad1-aaf8-e280757b7924"
+				(path "/1c02f793-f381-44cb-838a-dbb787484d0c/e61b723f-f359-4114-beb0-b4d2930b2aa9/5dfd95b7-fa55-40ea-ba4a-f8cc81696003"
+					(reference "C4")
+					(unit 1)
+				)
+				(path "/1c02f793-f381-44cb-838a-dbb787484d0c/e61b723f-f359-4114-beb0-b4d2930b2aa9/78dabe0b-e431-4181-9be1-9ea04483a27d"
 					(reference "C5")
-					(unit 1)
-				)
-				(path "/1c02f793-f381-44cb-838a-dbb787484d0c/e61b723f-f359-4114-beb0-b4d2930b2aa9/8611289c-07e1-4e14-a4ca-43f16a4333a9"
-					(reference "C4")
 					(unit 1)
 				)
@@
 			)
 		)
+		(property "LCSC" "C5349959"
+			(at 140.97 50.8 0)
+			(effects
+				(font
+					(size 1.27 1.27)
+				)
+				(hide yes)
+			)
+		)
 		(pin "6"
 		)
@@
 		(instances
 			(project "target"
-				(path "/1c02f793-f381-44cb-838a-dbb787484d0c/e61b723f-f359-4114-beb0-b4d2930b2aa9/560cd6ce-e08c-4984-ad6c-35893396417e"
-					(reference "D11")
-					(unit 1)
-				)
-				(path "/1c02f793-f381-44cb-838a-dbb787484d0c/e61b723f-f359-4114-beb0-b4d2930b2aa9/7ee20812-a607-4ad1-aaf8-e280757b7924"
-					(reference "D19")
-					(unit 1)
-				)
-				(path "/1c02f793-f381-44cb-838a-dbb787484d0c/e61b723f-f359-4114-beb0-b4d2930b2aa9/8611289c-07e1-4e14-a4ca-43f16a4333a9"
+				(path "/1c02f793-f381-44cb-838a-dbb787484d0c/e61b723f-f359-4114-beb0-b4d2930b2aa9/2577de81-7bff-4af3-a196-645474f5bc39"
+					(reference "D9")
+					(unit 1)
+				)
+				(path "/1c02f793-f381-44cb-838a-dbb787484d0c/e61b723f-f359-4114-beb0-b4d2930b2aa9/5dfd95b7-fa55-40ea-ba4a-f8cc81696003"
+					(reference "D13")
+					(unit 1)
+				)
+				(path "/1c02f793-f381-44cb-838a-dbb787484d0c/e61b723f-f359-4114-beb0-b4d2930b2aa9/78dabe0b-e431-4181-9be1-9ea04483a27d"
 					(reference "D17")
 					(unit 1)
@@
 			)
 		)
+		(property "LCSC" ""
+			(at 67.31 50.8 0)
+			(effects
+				(font
+					(size 1.27 1.27)
+				)
+				(hide yes)
+			)
+		)
 		(pin "3"
 		)
@@
 		(instances
 			(project "target"
-				(path "/1c02f793-f381-44cb-838a-dbb787484d0c/e61b723f-f359-4114-beb0-b4d2930b2aa9/560cd6ce-e08c-4984-ad6c-35893396417e"
+				(path "/1c02f793-f381-44cb-838a-dbb787484d0c/e61b723f-f359-4114-beb0-b4d2930b2aa9/2577de81-7bff-4af3-a196-645474f5bc39"
 					(reference "J12")
 					(unit 1)
 				)
-				(path "/1c02f793-f381-44cb-838a-dbb787484d0c/e61b723f-f359-4114-beb0-b4d2930b2aa9/7ee20812-a607-4ad1-aaf8-e280757b7924"
+				(path "/1c02f793-f381-44cb-838a-dbb787484d0c/e61b723f-f359-4114-beb0-b4d2930b2aa9/5dfd95b7-fa55-40ea-ba4a-f8cc81696003"
+					(reference "J16")
+					(unit 1)
+				)
+				(path "/1c02f793-f381-44cb-838a-dbb787484d0c/e61b723f-f359-4114-beb0-b4d2930b2aa9/78dabe0b-e431-4181-9be1-9ea04483a27d"
 					(reference "J20")
-					(unit 1)
-				)
-				(path "/1c02f793-f381-44cb-838a-dbb787484d0c/e61b723f-f359-4114-beb0-b4d2930b2aa9/8611289c-07e1-4e14-a4ca-43f16a4333a9"
-					(reference "J18")
 					(unit 1)
 				)
@@
 			)
 		)
+		(property "LCSC" ""
+			(at 181.61 50.8 0)
+			(effects
+				(font
+					(size 1.27 1.27)
+				)
+				(hide yes)
+			)
+		)
 		(pin "3"
 		)
@@
 		(instances
 			(project "target"
-				(path "/1c02f793-f381-44cb-838a-dbb787484d0c/e61b723f-f359-4114-beb0-b4d2930b2aa9/560cd6ce-e08c-4984-ad6c-35893396417e"
+				(path "/1c02f793-f381-44cb-838a-dbb787484d0c/e61b723f-f359-4114-beb0-b4d2930b2aa9/2577de81-7bff-4af3-a196-645474f5bc39"
 					(reference "J13")
 					(unit 1)
 				)
-				(path "/1c02f793-f381-44cb-838a-dbb787484d0c/e61b723f-f359-4114-beb0-b4d2930b2aa9/7ee20812-a607-4ad1-aaf8-e280757b7924"
+				(path "/1c02f793-f381-44cb-838a-dbb787484d0c/e61b723f-f359-4114-beb0-b4d2930b2aa9/5dfd95b7-fa55-40ea-ba4a-f8cc81696003"
+					(reference "J17")
+					(unit 1)
+				)
+				(path "/1c02f793-f381-44cb-838a-dbb787484d0c/e61b723f-f359-4114-beb0-b4d2930b2aa9/78dabe0b-e431-4181-9be1-9ea04483a27d"
 					(reference "J21")
-					(unit 1)
-				)
-				(path "/1c02f793-f381-44cb-838a-dbb787484d0c/e61b723f-f359-4114-beb0-b4d2930b2aa9/8611289c-07e1-4e14-a4ca-43f16a4333a9"
-					(reference "J19")
 					(unit 1)
 				)
@@
 			)
 		)
+		(property "LCSC" "C5349959"
+			(at 102.87 50.8 0)
+			(effects
+				(font
+					(size 1.27 1.27)
+				)
+				(hide yes)
+			)
+		)
 		(pin "6"
 		)
@@
 		(instances
 			(project "target"
-				(path "/1c02f793-f381-44cb-838a-dbb787484d0c/e61b723f-f359-4114-beb0-b4d2930b2aa9/560cd6ce-e08c-4984-ad6c-35893396417e"
-					(reference "D10")
-					(unit 1)
-				)
-				(path "/1c02f793-f381-44cb-838a-dbb787484d0c/e61b723f-f359-4114-beb0-b4d2930b2aa9/7ee20812-a607-4ad1-aaf8-e280757b7924"
-					(reference "D18")
-					(unit 1)
-				)
-				(path "/1c02f793-f381-44cb-838a-dbb787484d0c/e61b723f-f359-4114-beb0-b4d2930b2aa9/8611289c-07e1-4e14-a4ca-43f16a4333a9"
+				(path "/1c02f793-f381-44cb-838a-dbb787484d0c/e61b723f-f359-4114-beb0-b4d2930b2aa9/2577de81-7bff-4af3-a196-645474f5bc39"
+					(reference "D8")
+					(unit 1)
+				)
+				(path "/1c02f793-f381-44cb-838a-dbb787484d0c/e61b723f-f359-4114-beb0-b4d2930b2aa9/5dfd95b7-fa55-40ea-ba4a-f8cc81696003"
+					(reference "D12")
+					(unit 1)
+				)
+				(path "/1c02f793-f381-44cb-838a-dbb787484d0c/e61b723f-f359-4114-beb0-b4d2930b2aa9/78dabe0b-e431-4181-9be1-9ea04483a27d"
 					(reference "D16")
 					(unit 1)

Commit message: finished all pcbs by adjusting traces acording to 1oz copper weight
Parts:
- J6, J7: now left out of the parts list
Changed lines of the file:
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@@
 		(unit 1)
 		(exclude_from_sim no)
-		(in_bom yes)
+		(in_bom no)
 		(on_board yes)
 		(dnp no)
@@
 		(unit 1)
 		(exclude_from_sim no)
-		(in_bom yes)
+		(in_bom no)
 		(on_board yes)
 		(dnp no)
